File: lipo_drainer_schematic/lipo_drainer_schematic.kicad_sch (KiCad schematic)
At the start: 58 parts, among them J1 BATT, J2 FAN, J3 Vcal, J4 128x64_OLED, J5 Gcal, J6 Ical, J7 Heatsink Temp (for MCP7901), Q1 MMBT3904, Q10 G700P06T, Q11 G700P06T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

Commit message: Label cleanup
Parts:
- J7: value Heatsink Temp (for MCP7901) -> MCP7901; footprint Connector_PinHeader_2.54mm:PinHeader_1x03_P2.54mm_Vertical -> Package_TO_SOT_THT:TO-92_Inline; symbol Connector:Conn_01x03_Pin -> Sensor_Temperature:LM35-LP
Connections:
- net 3V3: now also J7.1 (+V_{S}); no longer J7.2 (Pin_2)
- net GND: now also J7.3 (GND); no longer J7.1 (Pin_1)
- net TEMP: now also J7.2 (V_{OUT}); no longer J7.3 (Pin_3)
Changed lines of the file:
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@@
     (stroke (width 0) (type default))
   )
-  (wire (pts (xy 150.495 90.17) (xy 150.495 133.35))
+  (wire (pts (xy 150.495 90.17) (xy 150.495 125.095))
     (stroke (width 0) (type default))
   )
@@
     (stroke (width 0) (type default))
   )
-  (wire (pts (xy 150.495 135.89) (xy 154.94 135.89))
+  (wire (pts (xy 151.13 135.255) (xy 155.575 135.255))
     (stroke (width 0) (type default))
   )
@@
     (stroke (width 0) (type default))
   )
+  (wire (pts (xy 101.6 144.145) (xy 200.66 144.145))
+    (stroke (width 0) (type default))
+  )
   (polyline (pts (xy 255.27 64.77) (xy 255.27 71.755))
     (stroke (width 0) (type default))
@@
     (stroke (width 0) (type default))
   )
-  (wire (pts (xy 101.6 144.145) (xy 200.66 144.145))
-    (stroke (width 0) (type default))
-  )
   (wire (pts (xy 71.755 55.88) (xy 76.835 55.88))
     (stroke (width 0) (type default))
@@
     (stroke (width 0) (type default))
   )
-  (wire (pts (xy 150.495 133.35) (xy 154.94 133.35))
+  (wire (pts (xy 150.495 125.095) (xy 163.195 125.095))
     (stroke (width 0) (type default))
   )
@@
     (effects (font (size 1.27 1.27)) (justify left bottom))
   )
-  (label "TEMP" (at 150.495 133.35 0) (fields_autoplaced)
+  (label "TEMP" (at 150.495 125.095 0) (fields_autoplaced)
     (effects (font (size 1.27 1.27)) (justify left bottom))
   )
@@
     (effects (font (size 1.27 1.27)) (justify left bottom))
   )
-  (label "3V3" (at 150.495 135.89 0) (fields_autoplaced)
+  (label "3V3" (at 151.13 135.255 0) (fields_autoplaced)
     (effects (font (size 1.27 1.27)) (justify left bottom))
   )
@@
     )
   )
-  (symbol (lib_id "Connector:Conn_01x03_Pin") (at 160.02 135.89 180) (unit 1)
-    (in_bom yes) (on_board yes) (dnp no) (fields_autoplaced)
-    (property "Reference" "J7" (at 161.29 135.255 0)
+  (symbol (lib_id "Sensor_Temperature:LM35-LP") (at 163.195 135.255 90) (unit 1)
+    (in_bom yes) (on_board yes) (dnp no)
+    (property "Reference" "J7" (at 163.83 136.525 0)
       (effects (font (size 1.27 1.27)) (justify right))
     )
-    (property "Value" "Heatsink Temp (for MCP7901)" (at 161.29 137.795 0)
+    (property "Value" "MCP7901" (at 169.545 124.46 0)
       (effects (font (size 1.27 1.27)) (justify right))
     )
-    (property "Footprint" "Connector_PinHeader_2.54mm:PinHeader_1x03_P2.54mm_Vertical" (at 160.02 135.89 0)
-      (effects (font (size 1.27 1.27)) hide)
-    )
-    (property "Datasheet" "~" (at 160.02 135.89 0)
+    (property "Footprint" "Package_TO_SOT_THT:TO-92_Inline" (at 169.545 133.985 0)
+      (effects (font (size 1.27 1.27)) (justify left) hide)
+    )
+    (property "Datasheet" "http://www.ti.com/lit/ds/symlink/lm35.pdf" (at 163.195 135.255 0)
       (effects (font (size 1.27 1.27)) hide)
     )
@@
     )
   )
-  (symbol (lib_id "power:GND") (at 154.94 138.43 0) (unit 1)
+  (symbol (lib_id "power:GND") (at 170.815 135.255 0) (unit 1)
     (in_bom yes) (on_board yes) (dnp no) (fields_autoplaced)
-    (property "Reference" "#PWR026" (at 154.94 144.78 0)
-      (effects (font (size 1.27 1.27)) hide)
-    )
-    (property "Value" "GND" (at 154.94 142.875 0)
-      (effects (font (size 1.27 1.27)))
-    )
-    (property "Footprint" "" (at 154.94 138.43 0)
-      (effects (font (size 1.27 1.27)) hide)
-    )
-    (property "Datasheet" "" (at 154.94 138.43 0)
-      (effects (font (size 1.27 1.27)) hide)
-    )
+    (property "Reference" "#PWR026" (at 170.815 141.605 0)
+      (effects (font (size 1.27 1.27)) hide)
+    )
+    (property "Value" "GND" (at 170.815 139.7 0)
+      (effects (font (size 1.27 1.27)))
+    )
+    (property "Footprint" "" (at 170.815 135.255 0)
+      (effects (font (size 1.27 1.27)) hide)
+    )
+    (property "Datasheet" "" (at 170.815 135.255 0)
+      (effects (font (size 1.27 1.27)) hide)
+    )

Commit message: Changed OFF button to be directly connected to the FET
Parts:
- added R26: 100, Resistor_SMD:R_0805_2012Metric_Pad1.20x1.40mm_HandSolder, symbol Device:R
Connections:
- net BAT+: now also R26.2
- net GND: no longer SW1.2
- net OFF: now also Q2.1 (G), R2.2, R3.1; no longer U2.9 (GPIO6)
- new net: R26.1, SW1.2
- no-connect marks 19 -> 20
Changed lines of the file:
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@@
   (junction (at 158.115 87.63) (diameter 0) (color 0 0 0 0)
   )
-  (junction (at 60.325 151.13) (diameter 0) (color 0 0 0 0)
-  )
   (junction (at 256.54 108.585) (diameter 0) (color 0 0 0 0)
   )
@@
   (junction (at 238.76 86.995) (diameter 0) (color 0 0 0 0)
   )
+  (no_connect (at 106.68 95.25))
   (no_connect (at 106.68 74.93))
   (no_connect (at 106.68 85.09))
@@
     (stroke (width 0) (type default))
   )
-  (polyline (pts (xy 66.04 169.545) (xy 66.04 134.62))
+  (polyline (pts (xy 80.01 169.545) (xy 80.01 134.62))
     (stroke (width 0) (type default))
   )
@@
     (stroke (width 0) (type default))
   )
-  (polyline (pts (xy 41.91 169.545) (xy 66.04 169.545))
+  (polyline (pts (xy 41.91 169.545) (xy 80.01 169.545))
     (stroke (width 0) (type default))
   )
@@
     (stroke (width 0) (type default))
   )
+  (wire (pts (xy 71.755 142.24) (xy 77.47 142.24))
+    (stroke (width 0) (type default))
+  )
   (wire (pts (xy 203.2 146.685) (xy 203.2 142.875))
     (stroke (width 0) (type default))
@@
     (stroke (width 0) (type default))
   )
+  (wire (pts (xy 66.675 63.5) (xy 69.85 63.5))
+    (stroke (width 0) (type default))
+  )
   (wire (pts (xy 174.625 55.245) (xy 174.625 57.785))
     (stroke (width 0) (type default))
@@
     (stroke (width 0) (type default))
   )
-  (polyline (pts (xy 66.04 134.62) (xy 41.91 134.62))
+  (polyline (pts (xy 80.01 134.62) (xy 41.91 134.62))
     (stroke (width 0) (type default))
   )
@@
     (stroke (width 0) (type default))
   )
-  (wire (pts (xy 60.325 142.24) (xy 60.325 151.13))
-    (stroke (width 0) (type default))
-  )
   (wire (pts (xy 144.145 105.41) (xy 142.24 105.41))
     (stroke (width 0) (type default))
@@
     (stroke (width 0) (type default))
   )
-  (wire (pts (xy 102.87 95.25) (xy 106.68 95.25))
-    (stroke (width 0) (type default))
-  )
   (wire (pts (xy 56.515 55.88) (xy 61.595 55.88))
     (stroke (width 0) (type default))
@@
   )
   (polyline (pts (xy 240.665 93.98) (xy 240.665 84.455))
+    (stroke (width 0) (type default))
+  )
+  (wire (pts (xy 60.325 142.24) (xy 64.135 142.24))
     (stroke (width 0) (type default))
   )
@@
     (effects (font (size 1.27 1.27)) (justify left bottom))
   )
+  (label "OFF" (at 67.945 63.5 0) (fields_autoplaced)
+    (effects (font (size 1.27 1.27)) (justify left bottom))
+  )
   (label "SDA" (at 102.87 87.63 0) (fields_autoplaced)
     (effects (font (size 1.27 1.27)) (justify left bottom))
@@
     (effects (font (size 1.27 1.27)) (justify left bottom))
   )
+  (label "BAT+" (at 74.295 142.24 0) (fields_autoplaced)
+    (effects (font (size 1.27 1.27)) (justify left bottom))
+  )
   (label "BAT+" (at 53.975 27.305 0) (fields_autoplaced)
     (effects (font (size 1.27 1.27)) (justify left bottom))
@@
   )
   (label "FAN+" (at 145.415 162.56 0) (fields_autoplaced)
-    (effects (font (size 1.27 1.27)) (justify left bottom))
-  )
-  (label "OFF" (at 102.87 95.25 0) (fields_autoplaced)
     (effects (font (size 1.27 1.27)) (justify left bottom))
   )
@@
         )
       )
+    )
+  )
+  (symbol (lib_id "Device:R") (at 67.945 142.24 90) (unit 1)
+    (in_bom yes) (on_board yes) (dnp no)
+    (property "Reference" "R26" (at 67.945 139.7 90)
+      (effects (font (size 1.27 1.27)))
+    )
+    (property "Value" "100" (at 67.945 142.24 90)
+      (effects (font (size 1.27 1.27)))
+    )
+    (property "Footprint" "Resistor_SMD:R_0805_2012Metric_Pad1.20x1.40mm_HandSolder" (at 67.945 144.018 90)
+      (effects (font (size 1.27 1.27)) hide)
+    )
+    (property "Datasheet" "~" (at 67.945 142.24 0)
+      (effects (font (size 1.27 1.27)) hide)
+    )
+    (pin "1")
+    (pin "2")
+    (instances
+      (project "lipo_drainer_schematic"
+        (path "/db6692d0-0595-40e8-a350-9f6ef4d6e67d"
+          (reference "R26") (unit 1)
+        )
+      )

Commit message: Added Zener inductance protection.
Parts:
- added D3: 1N5363BG, Diode_THT:D_DO-201AD_P15.24mm_Horizontal, symbol Diode:1N47xxA
Connections:
- net BAT+: now also D3.1 (K)
- net GND: now also D3.2 (A)
Changed lines of the file:
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@@
   (junction (at 158.115 87.63) (diameter 0) (color 0 0 0 0)
   )
+  (junction (at 34.29 27.305) (diameter 0) (color 0 0 0 0)
+  )
   (junction (at 256.54 108.585) (diameter 0) (color 0 0 0 0)
   )
@@
   )
   (junction (at 138.43 170.18) (diameter 0) (color 0 0 0 0)
+  )
+  (junction (at 29.21 34.925) (diameter 0) (color 0 0 0 0)
   )
   (junction (at 262.255 108.585) (diameter 0) (color 0 0 0 0)
@@
     (stroke (width 0) (type default))
   )
-  (wire (pts (xy 29.21 27.305) (xy 56.515 27.305))
-    (stroke (width 0) (type default))
-  )
   (wire (pts (xy 127 43.815) (xy 165.1 43.815))
     (stroke (width 0) (type default))
@@
     (stroke (width 0) (type default))
   )
+  (wire (pts (xy 29.21 27.305) (xy 34.29 27.305))
+    (stroke (width 0) (type default))
+  )
   (polyline (pts (xy 193.675 64.77) (xy 193.675 93.98))
     (stroke (width 0) (type default))
@@
     (stroke (width 0) (type default))
   )
-  (polyline (pts (xy 18.415 41.91) (xy 31.115 41.91))
+  (polyline (pts (xy 18.415 41.91) (xy 45.085 41.91))
     (stroke (width 0) (type default))
   )
@@
     (stroke (width 0) (type default))
   )
-  (polyline (pts (xy 31.115 41.91) (xy 31.115 29.845))
-    (stroke (width 0) (type default))
-  )
   (wire (pts (xy 238.76 84.455) (xy 238.76 86.995))
     (stroke (width 0) (type default))
@@
     (stroke (width 0) (type default))
   )
-  (polyline (pts (xy 18.415 22.225) (xy 38.1 22.225))
+  (polyline (pts (xy 18.415 22.225) (xy 45.085 22.225))
     (stroke (width 0) (type default))
   )
@@
     (stroke (width 0) (type default))
   )
-  (polyline (pts (xy 38.1 29.845) (xy 38.1 22.225))
+  (polyline (pts (xy 45.085 41.91) (xy 45.085 22.225))
     (stroke (width 0) (type default))
   )
@@
     (stroke (width 0) (type default))
   )
+  (wire (pts (xy 29.21 34.925) (xy 34.29 34.925))
+    (stroke (width 0) (type default))
+  )
   (wire (pts (xy 92.71 105.41) (xy 92.71 118.11))
     (stroke (width 0) (type default))
@@
     (stroke (width 0) (type default))
   )
+  (wire (pts (xy 34.29 27.305) (xy 56.515 27.305))
+    (stroke (width 0) (type default))
+  )
   (polyline (pts (xy 168.91 46.355) (xy 189.23 46.355))
     (stroke (width 0) (type default))
@@
   )
   (wire (pts (xy 147.955 115.57) (xy 238.125 115.57))
-    (stroke (width 0) (type default))
-  )
-  (polyline (pts (xy 31.115 29.845) (xy 38.1 29.845))
     (stroke (width 0) (type default))
   )
@@
         )
       )
+    )
+  )
+  (symbol (lib_id "Diode:1N47xxA") (at 34.29 31.115 270) (unit 1)
+    (in_bom yes) (on_board yes) (dnp no)
+    (property "Reference" "D3" (at 36.83 30.48 90)
+      (effects (font (size 1.27 1.27)) (justify left))
+    )
+    (property "Value" "1N5363BG" (at 33.02 36.83 90)
+      (effects (font (size 1.27 1.27)) (justify left))
+    )
+    (property "Footprint" "Diode_THT:D_DO-201AD_P15.24mm_Horizontal" (at 29.845 31.115 0)
+      (effects (font (size 1.27 1.27)) hide)
+    )
+    (property "Datasheet" "https://www.onsemi.com/pdf/datasheet/1n5333b-d.pdf" (at 34.29 31.115 0)
+      (effects (font (size 1.27 1.27)) hide)
+    )
+    (pin "1")
+    (pin "2")
+    (instances
+      (project "lipo_drainer_schematic"
+        (path "/db6692d0-0595-40e8-a350-9f6ef4d6e67d"
+          (reference "D3") (unit 1)
+        )
+      )

Commit message: Added motor BJT pulldown and redid ground planes
Parts:
- added R27: 50k, Resistor_SMD:R_0805_2012Metric_Pad1.20x1.40mm_HandSolder, symbol Device:R
Connections:
- net GND: now also R27.1
- net at Q4.1 (B), R4.2: now also R27.2
Other:
- moved on the sheet: D1, J2, Q3, Q4, R4, R5, R6

Commit message: Changed fan to PWMs
Parts:
- removed Q3: SiA469DJ, Package_TO_SOT_SMD:Vishay_PowerPAK_SC70-6L_Single, symbol Transistor_FET:SiA449DJ
- removed Q4: MMBT3904, Package_TO_SOT_SMD:SOT-23, symbol Transistor_BJT:MMBT3904
- removed R27: 50k, Resistor_SMD:R_0805_2012Metric_Pad1.20x1.40mm_HandSolder, symbol Device:R
- removed R4: 1k, Resistor_SMD:R_0805_2012Metric_Pad1.20x1.40mm_HandSolder, symbol Device:R
- removed R5: 100, Resistor_SMD:R_0805_2012Metric_Pad1.20x1.40mm_HandSolder, symbol Device:R
- removed R6: 5k, Resistor_SMD:R_0805_2012Metric_Pad1.20x1.40mm_HandSolder, symbol Device:R
- added J8: FAN2, Connector_PinSocket_2.54mm:PinSocket_1x02_P2.54mm_Vertical, symbol Connector:Conn_01x04_Pin
- added U1: MC7812BDTG, Package_TO_SOT_SMD:TO-252-2, symbol Regulator_Linear:NVC8674DS120
- J2: value FAN -> FAN1; symbol Connector:Conn_01x02_Pin -> Connector:Conn_01x04_Pin
Connections:
- net BAT+: now also U1.1 (IN)
- net FAN: now also J2.4 (Pin_4), J8.4 (Pin_4)
- net FAN+: now also J8.2 (Pin_2), U1.3 (OUT)
- net GND: now also J8.1 (Pin_1), U1.2 (GND)
Other:
- moved on the sheet: D1

Commit message: Updated fuse holder
Parts:
- F1: value MHP-TAT18-9-90N -> 40A Glass; footprint Fuse:Fuse_Schurter_UMZ250 -> Fuse:Fuseholder_Clip-6.3x32mm_Littelfuse_102_Inline_P34.21x7.62mm_D2.54mm_Horizontal
Connections:
- no-connect marks 20 -> 22
Changed lines of the file:
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@@
   (no_connect (at 106.68 123.19))
   (no_connect (at 106.68 77.47))
+  (no_connect (at 159.385 166.37))
   (no_connect (at 83.185 58.42))
   (no_connect (at 142.24 102.87))
@@
   (no_connect (at 106.68 113.03))
   (no_connect (at 142.24 82.55))
+  (no_connect (at 147.32 166.37))
   (no_connect (at 142.24 74.93))
   (no_connect (at 121.92 128.27))
@@
       (effects (font (size 1.27 1.27)))
     )
-    (property "Value" "MHP-TAT18-9-90N" (at 180.975 24.13 90)
-      (effects (font (size 1.27 1.27)))
-    )
-    (property "Footprint" "Fuse:Fuse_Schurter_UMZ250" (at 180.975 29.083 90)
-      (effects (font (size 1.27 1.27)) hide)
-    )
-    (property "Datasheet" "~" (at 180.975 27.305 0)
-      (effects (font (size 1.27 1.27)) hide)
-    )
+    (property "Value" "40A Glass" (at 180.975 24.13 90)
+      (effects (font (size 1.27 1.27)))
+    )
+    (property "Footprint" "Fuse:Fuseholder_Clip-6.3x32mm_Littelfuse_102_Inline_P34.21x7.62mm_D2.54mm_Horizontal" (at 180.975 29.083 90)
+      (effects (font (size 1.27 1.27)) hide)
+    )
+    (property "Datasheet" "https://www.digikey.com/en/products/detail/littelfuse-inc/0311030-M/3426887" (at 180.975 27.305 0)
+      (effects (font (size 1.27 1.27)) hide)
+    )
