File: lipo_drainer_schematic/lipo_drainer_schematic.kicad_sch (KiCad schematic)
At the start: 57 parts, among them J1 BATT, J2 FAN1, J3 Vcal, J4 128x64_OLED, J5 Gcal, J6 Ical, J7 MCP7901, J8 FAN2, Q1 MMBT3904, Q10 G700P06T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

Commit message: Updated PCB layout
Parts:
- added C5: 10u, Capacitor_SMD:C_1206_3216Metric_Pad1.33x1.80mm_HandSolder, symbol Device:C_Polarized
- added C6: 1u, Capacitor_SMD:C_1206_3216Metric_Pad1.33x1.80mm_HandSolder, symbol Device:C
- J2, J8: footprint Connector_PinSocket_2.54mm:PinSocket_1x02_P2.54mm_Vertical -> Connector_PinSocket_2.54mm:PinSocket_1x04_P2.54mm_Vertical
Connections:
- net BAT+: now also C6.1
- net FAN+: now also C5.1
- net GND: now also C5.2, C6.2
Other:
- moved on the sheet: U1
Changed lines of the file:
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@@
   (junction (at 275.59 90.805) (diameter 0) (color 0 0 0 0)
   )
+  (junction (at 77.47 27.305) (diameter 0) (color 0 0 0 0)
+  )
   (junction (at 177.165 102.235) (diameter 0) (color 0 0 0 0)
   )
@@
   (junction (at 174.625 67.945) (diameter 0) (color 0 0 0 0)
   )
+  (junction (at 109.855 168.275) (diameter 0) (color 0 0 0 0)
+  )
   (junction (at 247.015 100.965) (diameter 0) (color 0 0 0 0)
   )
@@
   (junction (at 238.76 86.995) (diameter 0) (color 0 0 0 0)
   )
+  (junction (at 129.54 168.275) (diameter 0) (color 0 0 0 0)
+  )
   (no_connect (at 106.68 95.25))
   (no_connect (at 106.68 74.93))
@@
     (stroke (width 0) (type default))
   )
+  (wire (pts (xy 77.47 27.305) (xy 167.64 27.305))
+    (stroke (width 0) (type default))
+  )
   (polyline (pts (xy 193.675 93.98) (xy 240.665 93.98))
     (stroke (width 0) (type default))
@@
     (stroke (width 0) (type default))
   )
-  (wire (pts (xy 56.515 27.305) (xy 167.64 27.305))
+  (wire (pts (xy 56.515 27.305) (xy 77.47 27.305))
     (stroke (width 0) (type default))
   )
@@
     (stroke (width 0) (type default))
   )
+  (wire (pts (xy 129.54 168.275) (xy 137.795 168.275))
+    (stroke (width 0) (type default))
+  )
   (polyline (pts (xy 217.17 147.32) (xy 245.745 147.32))
     (stroke (width 0) (type default))
@@
     (stroke (width 0) (type default))
   )
+  (wire (pts (xy 109.855 168.275) (xy 113.03 168.275))
+    (stroke (width 0) (type default))
+  )
   (wire (pts (xy 142.24 90.17) (xy 150.495 90.17))
     (stroke (width 0) (type default))
@@
     (stroke (width 0) (type default))
   )
-  (wire (pts (xy 99.695 168.275) (xy 118.745 168.275))
+  (wire (pts (xy 93.98 168.275) (xy 109.855 168.275))
     (stroke (width 0) (type default))
   )
@@
     (stroke (width 0) (type default))
   )
-  (wire (pts (xy 133.985 168.275) (xy 137.795 168.275))
+  (wire (pts (xy 128.27 168.275) (xy 129.54 168.275))
     (stroke (width 0) (type default))
   )
@@
     (stroke (width 0) (type default))
   )
-  (rectangle (start 111.76 151.765) (end 167.64 188.595)
+  (rectangle (start 102.235 151.765) (end 167.64 188.595)
     (stroke (width 0) (type default))
     (fill (type none))
@@
     (effects (font (size 1.27 1.27)) (justify left bottom))
   )
-  (label "BAT+" (at 104.14 168.275 0) (fields_autoplaced)
+  (label "BAT+" (at 97.79 168.275 0) (fields_autoplaced)
     (effects (font (size 1.27 1.27)) (justify left bottom))
   )
@@
     )
   )
+  (symbol (lib_id "power:GND") (at 129.54 175.895 0) (unit 1)
+    (in_bom yes) (on_board yes) (dnp no) (fields_autoplaced)
+    (property "Reference" "#PWR030" (at 129.54 182.245 0)
+      (effects (font (size 1.27 1.27)) hide)
+    )
+    (property "Value" "GND" (at 129.54 180.34 0)
+      (effects (font (size 1.27 1.27)))
+    )
+    (property "Footprint" "" (at 129.54 175.895 0)
+      (effects (font (size 1.27 1.27)) hide)
+    )
+    (property "Datasheet" "" (at 129.54 175.895 0)
+      (effects (font (size 1.27 1.27)) hide)
+    )
+    (pin "1")
+    (instances
+      (project "lipo_drainer_schematic"
+        (path "/db6692d0-0595-40e8-a350-9f6ef4d6e67d"
+          (reference "#PWR030") (unit 1)
+        )
+      )
+    )
+  )
   (symbol (lib_id "Device:R") (at 223.52 83.185 180) (unit 1)
     (in_bom yes) (on_board yes) (dnp no)
@@
     )
   )
+  (symbol (lib_id "Device:C") (at 109.855 172.085 0) (unit 1)
+    (in_bom yes) (on_board yes) (dnp no)
+    (property "Reference" "C6" (at 106.68 170.18 0)
+      (effects (font (size 1.27 1.27)) (justify left))
+    )
+    (property "Value" "1u" (at 104.775 174.625 0)
+      (effects (font (size 1.27 1.27)) (justify left))
+    )
+    (property "Footprint" "Capacitor_SMD:C_1206_3216Metric_Pad1.33x1.80mm_HandSolder" (at 110.8202 175.895 0)
+      (effects (font (size 1.27 1.27)) hide)
+    )
+    (property "Datasheet" "~" (at 109.855 172.085 0)
+      (effects (font (size 1.27 1.27)) hide)
+    )
+    (pin "1")
+    (pin "2")
+    (instances
+      (project "lipo_drainer_schematic"
+        (path "/db6692d0-0595-40e8-a350-9f6ef4d6e67d"
+          (reference "C6") (unit 1)
+        )
+      )
+    )
+  )
   (symbol (lib_id "Reference_Voltage:LM4040DBZ-3") (at 247.015 104.775 90) (unit 1)
     (in_bom yes) (on_board yes) (dnp no)
@@
     )
   )
+  (symbol (lib_id "Device:C_Polarized") (at 129.54 172.085 0) (unit 1)
+    (in_bom yes) (on_board yes) (dnp no) (fields_autoplaced)
+    (property "Reference" "C5" (at 133.35 169.9259 0)
+      (effects (font (size 1.27 1.27)) (justify left))
+    )
+    (property "Value" "10u" (at 133.35 172.4659 0)
+      (effects (font (size 1.27 1.27)) (justify left))
+    )
+    (property "Footprint" "Capacitor_SMD:C_1206_3216Metric_Pad1.33x1.80mm_HandSolder" (at 130.5052 175.895 0)
+      (effects (font (size 1.27 1.27)) hide)
+    )
+    (property "Datasheet" "~" (at 129.54 172.085 0)
+      (effects (font (size 1.27 1.27)) hide)
+    )
+    (pin "1")
+    (pin "2")
+    (instances
+      (project "lipo_drainer_schematic"
+        (path "/db6692d0-0595-40e8-a350-9f6ef4d6e67d"
+          (reference "C5") (unit 1)
+        )
+      )
+    )
+  )
   (symbol (lib_id "power:GND") (at 144.145 130.175 0) (unit 1)
     (in_bom yes) (on_board yes) (dnp no)
@@
     )
   )
-  (symbol (lib_id "Regulator_Linear:NVC8674DS120") (at 126.365 168.275 0) (unit 1)
+  (symbol (lib_id "Regulator_Linear:NVC8674DS120") (at 120.65 168.275 0) (unit 1)
     (in_bom yes) (on_board yes) (dnp no)
-    (property "Reference" "U1" (at 126.365 161.925 0)
+    (property "Reference" "U1" (at 120.65 161.925 0)
       (effects (font (size 1.27 1.27)))
     )
-    (property "Value" "MC7812BDTG" (at 126.365 164.465 0)
+    (property "Value" "MC7812BDTG" (at 120.65 164.465 0)
       (effects (font (size 1.27 1.27)))
     )
-    (property "Footprint" "Package_TO_SOT_SMD:TO-252-2" (at 126.365 168.275 0)
+    (property "Footprint" "Package_TO_SOT_SMD:TO-252-2" (at 120.65 168.275 0)
       (effects (font (size 1.27 1.27)) hide)
     )
-    (property "Datasheet" "https://www.onsemi.com/pdf/datasheet/mc7800-d.pdf" (at 126.365 168.275 0)
+    (property "Datasheet" "https://www.onsemi.com/pdf/datasheet/mc7800-d.pdf" (at 120.65 168.275 0)
       (effects (font (size 1.27 1.27)) hide)
     )
@@
       (effects (font (size 1.27 1.27)) (justify right))
     )
-    (property "Footprint" "Connector_PinSocket_2.54mm:PinSocket_1x02_P2.54mm_Vertical" (at 161.925 161.29 0)
+    (property "Footprint" "Connector_PinSocket_2.54mm:PinSocket_1x04_P2.54mm_Vertical" (at 161.925 161.29 0)
       (effects (font (size 1.27 1.27)) hide)
     )
@@
     )
   )
+  (symbol (lib_id "power:GND") (at 109.855 175.895 0) (unit 1)
+    (in_bom yes) (on_board yes) (dnp no) (fields_autoplaced)
+    (property "Reference" "#PWR031" (at 109.855 182.245 0)
+      (effects (font (size 1.27 1.27)) hide)
+    )
+    (property "Value" "GND" (at 109.855 180.34 0)
+      (effects (font (size 1.27 1.27)))
+    )
+    (property "Footprint" "" (at 109.855 175.895 0)
+      (effects (font (size 1.27 1.27)) hide)
+    )
+    (property "Datasheet" "" (at 109.855 175.895 0)
+      (effects (font (size 1.27 1.27)) hide)
+    )
+    (pin "1")
+    (instances
+      (project "lipo_drainer_schematic"
+        (path "/db6692d0-0595-40e8-a350-9f6ef4d6e67d"
+          (reference "#PWR031") (unit 1)
+        )
+      )
+    )
+  )
   (symbol (lib_id "power:GND") (at 152.4 172.72 0) (unit 1)
     (in_bom yes) (on_board yes) (dnp no) (fields_autoplaced)
@@
       (effects (font (size 1.27 1.27)) (justify right))
     )
-    (property "Footprint" "Connector_PinSocket_2.54mm:PinSocket_1x02_P2.54mm_Vertical" (at 149.86 161.29 0)
+    (property "Footprint" "Connector_PinSocket_2.54mm:PinSocket_1x04_P2.54mm_Vertical" (at 149.86 161.29 0)
       (effects (font (size 1.27 1.27)) hide)
     )
@@
     )
   )
-  (symbol (lib_id "power:GND") (at 126.365 175.895 0) (unit 1)
+  (symbol (lib_id "power:GND") (at 120.65 175.895 0) (unit 1)
     (in_bom yes) (on_board yes) (dnp no) (fields_autoplaced)
-    (property "Reference" "#PWR027" (at 126.365 182.245 0)
+    (property "Reference" "#PWR027" (at 120.65 182.245 0)
       (effects (font (size 1.27 1.27)) hide)
     )
-    (property "Value" "GND" (at 126.365 180.34 0)
+    (property "Value" "GND" (at 120.65 180.34 0)
       (effects (font (size 1.27 1.27)))
     )
-    (property "Footprint" "" (at 126.365 175.895 0)
+    (property "Footprint" "" (at 120.65 175.895 0)
       (effects (font (size 1.27 1.27)) hide)
     )
-    (property "Datasheet" "" (at 126.365 175.895 0)
+    (property "Datasheet" "" (at 120.65 175.895 0)
       (effects (font (size 1.27 1.27)) hide)
     )
@@
         )
       )
+    )
+  )
+  (symbol (lib_id "power:PWR_FLAG") (at 77.47 27.305 0) (unit 1)
+    (in_bom yes) (on_board yes) (dnp no) (fields_autoplaced)
+    (property "Reference" "#FLG04" (at 77.47 25.4 0)
+      (effects (font (size 1.27 1.27)) hide)
+    )
+    (property "Value" "PWR_FLAG" (at 77.47 23.495 0)
+      (effects (font (size 1.27 1.27)))
+    )
+    (property "Footprint" "" (at 77.47 27.305 0)
+      (effects (font (size 1.27 1.27)) hide)
+    )
+    (property "Datasheet" "~" (at 77.47 27.305 0)
+      (effects (font (size 1.27 1.27)) hide)
+    )
+    (pin "1")
+    (instances
+      (project "lipo_drainer_schematic"
+        (path "/db6692d0-0595-40e8-a350-9f6ef4d6e67d"
+          (reference "#FLG04") (unit 1)
+        )
+      )

Commit message: Added some UI to readme
Parts:
- C1, C2, C3, C4, C5, C6: digikey (none) -> https://www.digikey.com/en/products/detail/samsung-electro-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
- D1: digikey (none) -> https://www.digikey.com/en/products/detail/smc-diode-soluti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
- D3: digikey (none) -> https://www.digikey.com/en/products/detail/onsemi/1N5363BG/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
- F1: digikey (none) -> https://www.digikey.com/en/products/detail/littelfuse-inc/0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
- J1, J2, J3, J5, J6, J8: digikey (none) -> -
- J4: digikey (none) -> https://www.amazon.com/dp/B08V97FYD2/?coliid=I2KB2LA2D4KFSX
- J7: digikey (none) -> https://www.digikey.com/en/products/detail/microchip-techno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
- Q1, Q6, Q9: digikey (none) -> https://www.digikey.com/en/products/detail/onsemi/MMBT3904L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
- Q10, Q11, Q7, Q8: digikey (none) -> https://www.digikey.com/en/products/detail/goford-semicondu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
- Q2, Q5: digikey (none) -> https://www.digikey.com/en/products/detail/infineon-technol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
- R1: value 2k -> 2.2k; digikey (none) -> https://www.digikey.com/en/products/detail/panasonic-electr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
- R10, R11, R13, R15, R17, R19, R2, R20, R21, R25, R26, R7, R8, R9: digikey (none) -> https://www.digikey.com/en/products/detail/panasonic-electr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
- R12, R14, R18: value 50k -> 47k; digikey (none) -> https://www.digikey.com/en/products/detail/panasonic-electr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
- R16: value 5k -> 6.8k; digikey (none) -> https://www.digikey.com/en/products/detail/panasonic-electr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
- R22, R23, R24: digikey (none) -> https://www.digikey.com/en/products/detail/bourns-inc/PWR22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
- R3: value 5K -> 2.2k; digikey (none) -> https://www.digikey.com/en/products/detail/panasonic-electr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
- SW1, SW2, SW3, SW4, SW5: digikey (none) -> https://www.digikey.com/en/products/detail/c-k/PTS636-SM50-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
- U1: digikey (none) -> https://www.digikey.com/en/products/detail/onsemi/MC7812BDT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
- U2: digikey (none) -> https://www.digikey.com/en/products/detail/raspberry-pi/SC0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
- U3: digikey (none) -> https://www.digikey.com/en/products/detail/texas-instrument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
- U4, U5: digikey (none) -> https://www.digikey.com/en/products/detail/diodes-incorpora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
