File: xt60_array/xt60_array.kicad_sch (KiCad schematic)
At the start: 1 part, among them J1 XT60_INPUT

Commit message: Finished schematic
Parts:
- added D1, D2, D3, D4, D5, D6: STPS30SM60SG-TR, Matt:TO-263-2_TabPin1_Alt, symbol Diode:1.5KExxA
- added J2, J3, J4, J5, J6, J7: XT-60, Connector_AMASS:AMASS_XT60-M_1x02_P7.20mm_Vertical, symbol Connector:Conn_01x02_Socket
Connections:
- net at J1.1 (Pin_1): now also J2.1 (Pin_1), J3.1 (Pin_1), J4.1 (Pin_1), J5.1 (Pin_1), J6.1 (Pin_1), J7.1 (Pin_1)
- net at J1.2 (Pin_2): now also D1.1 (A1), D2.1 (A1), D3.1 (A1), D4.1 (A1), D5.1 (A1), D6.1 (A1)
- new net: D4.2 (A2), J4.2 (Pin_2)
- new net: D2.2 (A2), J2.2 (Pin_2)
- new net: D1.2 (A2), J7.2 (Pin_2)
- new net: D5.2 (A2), J5.2 (Pin_2)
- new net: D3.2 (A2), J3.2 (Pin_2)
- new net: D6.2 (A2), J6.2 (Pin_2)
Other:
- moved on the sheet: J1

Commit message: Missed some files on the last commit
Connections:
- net VCC: now reaches D1.1 (A1), D2.1 (A1), D3.1 (A1), D4.1 (A1), D5.1 (A1), D6.1 (A1), J1.2 (Pin_2)
- net GND: now reaches J1.1 (Pin_1), J2.1 (Pin_1), J3.1 (Pin_1), J4.1 (Pin_1), J5.1 (Pin_1), J6.1 (Pin_1), J7.1 (Pin_1)
Changed lines of the file:
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@@
   (junction (at 106.68 120.65) (diameter 0) (color 0 0 0 0)
   )
+  (junction (at 83.82 130.81) (diameter 0) (color 0 0 0 0)
+  )
   (junction (at 78.74 104.14) (diameter 0) (color 0 0 0 0)
   )
+  (junction (at 90.17 130.81) (diameter 0) (color 0 0 0 0)
+  )
   (junction (at 78.74 113.665) (diameter 0) (color 0 0 0 0)
   )
@@
     (stroke (width 0) (type default))
   )
-  (wire (pts (xy 106.68 130.81) (xy 78.74 130.81))
+  (wire (pts (xy 106.68 130.81) (xy 90.17 130.81))
     (stroke (width 0) (type default))
   )
@@
     (stroke (width 0) (type default))
   )
+  (wire (pts (xy 83.82 130.81) (xy 90.17 130.81))
+    (stroke (width 0) (type default))
+  )
   (wire (pts (xy 78.74 104.14) (xy 76.2 104.14))
     (stroke (width 0) (type default))
@@
     (stroke (width 0) (type default))
   )
+  (wire (pts (xy 83.82 130.81) (xy 78.74 130.81))
+    (stroke (width 0) (type default))
+  )
   (wire (pts (xy 78.74 123.19) (xy 76.2 123.19))
     (stroke (width 0) (type default))
@@
     (stroke (width 0) (type default))
   )
+  (label "VCC" (at 102.87 73.025 0) (fields_autoplaced)
+    (effects (font (size 1.27 1.27)) (justify left bottom))
+  )
   (symbol (lib_id "Diode:1.5KExxA") (at 90.17 92.075 180) (unit 1)
     (in_bom yes) (on_board yes) (dnp no) (fields_autoplaced)
@@
     )
   )
+  (symbol (lib_id "power:PWR_FLAG") (at 83.82 130.81 0) (unit 1)
+    (in_bom yes) (on_board yes) (dnp no) (fields_autoplaced)
+    (property "Reference" "#FLG01" (at 83.82 128.905 0)
+      (effects (font (size 1.27 1.27)) hide)
+    )
+    (property "Value" "PWR_FLAG" (at 83.82 127 0)
+      (effects (font (size 1.27 1.27)))
+    )
+    (property "Footprint" "" (at 83.82 130.81 0)
+      (effects (font (size 1.27 1.27)) hide)
+    )
+    (property "Datasheet" "~" (at 83.82 130.81 0)
+      (effects (font (size 1.27 1.27)) hide)
+    )
+    (pin "1")
+    (instances
+      (project "xt60_array"
+        (path "/58412afb-6627-46b9-ac0b-395aa32013d4"
+          (reference "#FLG01") (unit 1)
+        )
+      )
+    )
+  )
   (symbol (lib_id "Connector:Conn_01x02_Socket") (at 71.12 85.09 180) (unit 1)
     (in_bom yes) (on_board yes) (dnp no) (fields_autoplaced)
@@
         )
       )
+    )
+  )
+  (symbol (lib_id "power:GND") (at 90.17 130.81 0) (unit 1)
+    (in_bom yes) (on_board yes) (dnp no) (fields_autoplaced)
+    (property "Reference" "#PWR01" (at 90.17 137.16 0)
+      (effects (font (size 1.27 1.27)) hide)
+    )
+    (property "Value" "GND" (at 90.17 135.89 0)
+      (effects (font (size 1.27 1.27)))
+    )
+    (property "Footprint" "" (at 90.17 130.81 0)
+      (effects (font (size 1.27 1.27)) hide)
+    )
+    (property "Datasheet" "" (at 90.17 130.81 0)
+      (effects (font (size 1.27 1.27)) hide)
+    )
+    (pin "1")
+    (instances
+      (project "xt60_array"
+        (path "/58412afb-6627-46b9-ac0b-395aa32013d4"
+          (reference "#PWR01") (unit 1)
+        )
+      )

Commit message: Added some UI to readme
Parts:
- D1, D2, D3, D4, D5, D6: digikey (none) -> https://www.digikey.com/en/products/detail/stmicroelectroni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
Changed lines of the file:
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@@
+      (effects (font (size 1.27 1.27)) hide)
+    )
+    (property "digikey" "https://www.digikey.com/en/products/detail/stmicroelectronics/STPS30SM60SG-TR/2827026" (at 90.17 92.075 0)
       (effects (font (size 1.27 1.27)) hide)
     )
@@
       (effects (font (size 1.27 1.27)) hide)
     )
+    (property "digikey" "" (at 71.12 113.665 0)
+      (effects (font (size 1.27 1.27)) hide)
+    )
     (pin "1")
     (pin "2")
@@
       (effects (font (size 1.27 1.27)) hide)
     )
+    (property "digikey" "https://www.digikey.com/en/products/detail/stmicroelectronics/STPS30SM60SG-TR/2827026" (at 90.17 111.125 0)
+      (effects (font (size 1.27 1.27)) hide)
+    )
     (pin "1")
     (pin "2")
@@
       (effects (font (size 1.27 1.27)) hide)
     )
+    (property "digikey" "https://www.digikey.com/en/products/detail/stmicroelectronics/STPS30SM60SG-TR/2827026" (at 90.17 120.65 0)
+      (effects (font (size 1.27 1.27)) hide)
+    )
     (pin "1")
     (pin "2")
@@
     )
     (property "Datasheet" "~" (at 71.12 85.09 0)
+      (effects (font (size 1.27 1.27)) hide)
+    )
+    (property "digikey" "" (at 71.12 85.09 0)
       (effects (font (size 1.27 1.27)) hide)
     )
@@
       (effects (font (size 1.27 1.27)) hide)
     )
+    (property "digikey" "" (at 71.12 94.615 0)
+      (effects (font (size 1.27 1.27)) hide)
+    )
     (pin "1")
     (pin "2")
@@
       (effects (font (size 1.27 1.27)) hide)
     )
+    (property "digikey" "https://www.digikey.com/en/products/detail/stmicroelectronics/STPS30SM60SG-TR/2827026" (at 90.17 101.6 0)
+      (effects (font (size 1.27 1.27)) hide)
+    )
     (pin "1")
     (pin "2")
@@
       (effects (font (size 1.27 1.27)) hide)
     )
+    (property "digikey" "" (at 71.12 104.14 0)
+      (effects (font (size 1.27 1.27)) hide)
+    )
     (pin "1")
     (pin "2")
@@
       (effects (font (size 1.27 1.27)) hide)
     )
+    (property "digikey" "https://www.digikey.com/en/products/detail/stmicroelectronics/STPS30SM60SG-TR/2827026" (at 90.17 82.55 0)
+      (effects (font (size 1.27 1.27)) hide)
+    )
     (pin "1")
     (pin "2")
@@
     )
     (property "Datasheet" "~" (at 111.76 130.81 0)
+      (effects (font (size 1.27 1.27)) hide)
+    )
+    (property "digikey" "" (at 111.76 130.81 0)
       (effects (font (size 1.27 1.27)) hide)
     )
@@
       (effects (font (size 1.27 1.27)) hide)
     )
+    (property "digikey" "https://www.digikey.com/en/products/detail/stmicroelectronics/STPS30SM60SG-TR/2827026" (at 90.17 73.025 0)
+      (effects (font (size 1.27 1.27)) hide)
+    )
     (pin "1")
     (pin "2")
@@
       (effects (font (size 1.27 1.27)) hide)
     )
+    (property "digikey" "" (at 71.12 123.19 0)
+      (effects (font (size 1.27 1.27)) hide)
+    )
     (pin "1")
     (pin "2")
@@
       (effects (font (size 1.27 1.27)) hide)
     )
+    (property "digikey" "" (at 71.12 75.565 0)
+      (effects (font (size 1.27 1.27)) hide)
+    )
